Commit message: [MODIFY] modified for livox mid360

File: gazebo_simulation/livox_laser_simulation/urdf/livox_mid360.xacro (robot description, xacro)
@@ -4,5 +4,5 @@
   <xacro:property name="laser_min_range" value="0.1"/>
   <xacro:property name="laser_max_range" value="200.0"/>
-  <xacro:property name="ros_topic" value="scan"/>
+  <xacro:property name="ros_topic" value="livox/lidar"/>
   <xacro:property name="samples" value="24000"/>
   <xacro:property name="downsample" value="1"/>
@@ -15,5 +15,5 @@
     </inertial>
   </xacro:macro>
-  <xacro:macro name="Livox_Mid_gazebo_sensor" params="visualize:=True update_rate:=10 resolution:=0.002 noise_mean:=0.0 noise_stddev:=0.01 name:=livox">
+  <xacro:macro name="Livox_Mid_gazebo_sensor" params="visualize:=True update_rate:=10 resolution:=0.002 noise_mean:=0.0 publish_pointcloud_type:=3 noise_stddev:=0.01 name:=livox">
     <gazebo reference="${name}">
       <sensor type="ray" name="laser_${name}">
@@ -84,6 +84,6 @@
     <xacro:Livox_Mid_gazebo_sensor name="${name}" visualize="${visualize}"/>
   </xacro:macro>
-    <xacro:Livox_Mid40 name="livox"/>
+    <xacro:Livox_Mid_gazebo_sensor name="livox"/>
   <xacro:include filename="$(find livox_laser_simulation)/urdf/robot_core.xacro"/>
-  <xacro:link_ddmr name="ddmr"/>
+  <!--xacro:link_ddmr name="ddmr"/-->
 </robot>

File: gazebo_simulation/livox_laser_simulation/urdf/robot_core.xacro (robot description, xacro)
@@ -59,5 +59,5 @@
         </inertial>
     </xacro:macro>
-    <xacro:macro name="Livox_Mid_gazebo_sensor" params="visualize:=True update_rate:=10 resolution:=0.002 noise_mean:=0.0 noise_stddev:=0.01 name:=livox">
+    <xacro:macro name="Livox_Mid_gazebo_sensor" params="visualize:=True update_rate:=10 resolution:=0.002  noise_mean:=0.0 noise_stddev:=0.01 name:=livox">
         <gazebo reference="${name}">
         <sensor type="ray" name="laser_${name}">

Commit message: [MODIFY]1006: using livox custom msg, need to add IMU

File: gazebo_simulation/livox_laser_simulation/urdf/livox_mid360.xacro (robot description, xacro)
@@ -4,7 +4,8 @@
   <xacro:property name="laser_min_range" value="0.1"/>
   <xacro:property name="laser_max_range" value="200.0"/>
-  <xacro:property name="ros_topic" value="livox/lidar"/>
+  <xacro:property name="ros_topic" value="scan"/>
   <xacro:property name="samples" value="24000"/>
   <xacro:property name="downsample" value="1"/>
+  <xacro:property name="publish_pointcloud_type" value="3"/>
   <xacro:macro name="null_inertial">
     <inertial>
@@ -15,5 +16,5 @@
     </inertial>
   </xacro:macro>
-  <xacro:macro name="Livox_Mid_gazebo_sensor" params="visualize:=True update_rate:=10 resolution:=0.002 noise_mean:=0.0 publish_pointcloud_type:=3 noise_stddev:=0.01 name:=livox">
+  <xacro:macro name="Livox_Mid_gazebo_sensor" params="visualize:=True update_rate:=10 resolution:=0.002 noise_mean:=0.0 noise_stddev:=0.01 name:=livox">
     <gazebo reference="${name}">
       <sensor type="ray" name="laser_${name}">
@@ -54,4 +55,5 @@
 		  <csv_file_name>package://livox_laser_simulation/scan_mode/mid360.csv</csv_file_name>
 		  <ros_topic>${ros_topic}</ros_topic>
+      <publish_pointcloud_type>${publish_pointcloud_type}</publish_pointcloud_type>
         </plugin>
       </sensor>

File: gazebo_simulation/livox_laser_simulation/urdf/robot_core.xacro (robot description, xacro)
@@ -48,6 +48,7 @@
     <xacro:property name="laser_min_range" value="0.1"/>
     <xacro:property name="laser_max_range" value="200.0"/>
-    <xacro:property name="ros_topic" value="scan"/>
+    <xacro:property name="ros_topic" value="/livox/lidar"/>
     <xacro:property name="samples" value="24000"/>
+    <xacro:property name="publish_pointcloud_type" value="3"/>
     <xacro:property name="downsample" value="1"/>
     <xacro:macro name="null_inertial">
@@ -59,5 +60,5 @@
         </inertial>
     </xacro:macro>
-    <xacro:macro name="Livox_Mid_gazebo_sensor" params="visualize:=True update_rate:=10 resolution:=0.002  noise_mean:=0.0 noise_stddev:=0.01 name:=livox">
+    <xacro:macro name="Livox_Mid_gazebo_sensor" params="visualize:=True update_rate:=10 resolution:=0.002 noise_mean:=0.0 noise_stddev:=0.01 name:=livox">
         <gazebo reference="${name}">
         <sensor type="ray" name="laser_${name}">
@@ -98,4 +99,5 @@
             <csv_file_name>package://livox_laser_simulation/scan_mode/mid360.csv</csv_file_name>
             <ros_topic>${ros_topic}</ros_topic>
+            <publish_pointcloud_type>${publish_pointcloud_type}</publish_pointcloud_type>
             </plugin>
         </sensor>

Commit message: [ADD]nav, Fast-LIO mapping, Fast-LIO localization with gravity align added, .git file removed for integration

File: gazebo_simulation/livox_laser_simulation/urdf/livox_mid360.xacro (robot description, xacro)
@@ -3,5 +3,5 @@
   <xacro:property name="M_PI" value="3.14159"/>
   <xacro:property name="laser_min_range" value="0.1"/>
-  <xacro:property name="laser_max_range" value="200.0"/>
+  <xacro:property name="laser_max_range" value="20.0"/>
   <xacro:property name="ros_topic" value="scan"/>
   <xacro:property name="samples" value="24000"/>

File: gazebo_simulation/livox_laser_simulation/urdf/robot_core.xacro (robot description, xacro)
@@ -37,5 +37,5 @@
             </geometry>
         </collision>
-        <xacro:inertial_box mass="1.5" x="0.7" y="0.7" z="0.35">
+        <xacro:inertial_box mass="3.0" x="0.7" y="0.7" z="0.35">
             <origin xyz="0.35 0 0.175" rpy="0 0 0"/>
         </xacro:inertial_box>
@@ -47,5 +47,5 @@
     <xacro:property name="M_PI" value="3.14159"/>
     <xacro:property name="laser_min_range" value="0.1"/>
-    <xacro:property name="laser_max_range" value="200.0"/>
+    <xacro:property name="laser_max_range" value="20.0"/>
     <xacro:property name="ros_topic" value="/livox/lidar"/>
     <xacro:property name="samples" value="24000"/>
@@ -150,5 +150,5 @@
             </geometry>
         </collision>
-        <xacro:inertial_box mass="0.1" x="0.2" y="0.2" z="1.6">
+        <xacro:inertial_box mass="0.05" x="0.2" y="0.2" z="1.6">
             <origin xyz="0.0 0 0.8" rpy="0 0 0"/>
         </xacro:inertial_box>
@@ -160,5 +160,5 @@
 		<parent link="sensor_link"/>
 		<child link="livox_base"/>
-		<!-- <origin xyz="0.2 0 1.6" rpy="${M_PI/6} 0 0" /> -->
+		<!--origin xyz="0.2 0 1.6" rpy="${M_PI/6} 0 0" /-->
         <origin xyz="0.2 0 1.6" rpy="${M_PI/6} 0 ${M_PI/2}" />
 	</joint>
@@ -195,5 +195,5 @@
             </geometry>
         </collision>
-        <xacro:inertial_cylinder mass="0.5" length="0.05" radius="0.15">
+        <xacro:inertial_cylinder mass="1.0" length="0.05" radius="0.15">
             <origin xyz="0 0 0" rpy="0 0 0"/>
         </xacro:inertial_cylinder>
@@ -235,5 +235,5 @@
             </geometry>
         </collision>
-        <xacro:inertial_cylinder mass="0.5" length="0.05" radius="0.15">
+        <xacro:inertial_cylinder mass="1.0" length="0.05" radius="0.15">
             <origin xyz="0 0 0" rpy="0 0 0"/>
         </xacro:inertial_cylinder>
@@ -265,5 +265,5 @@
             </geometry>
         </collision>
-        <xacro:inertial_sphere mass="0.1" radius="0.15">
+        <xacro:inertial_sphere mass="0.5" radius="0.15">
             <origin xyz="0 0 0" rpy="0 0 0"/>
         </xacro:inertial_sphere>
@@ -291,5 +291,5 @@
             </geometry>
         </collision>
-        <xacro:inertial_sphere mass="0.1" radius="0.15">
+        <xacro:inertial_sphere mass="0.5" radius="0.15">
             <origin xyz="0 0 0" rpy="0 0 0"/>
         </xacro:inertial_sphere>
