Commit message: [MODIFY] gazebo sensor position modified, fast_lio_localization modified for tf input for move_base

File: gazebo_simulation/livox_laser_simulation/urdf/gazebo_control.xacro (robot description, xacro)
@@ -18,6 +18,6 @@
             <robot_base_frame>base_link</robot_base_frame>
             <publishWheelTF>true</publishWheelTF>
-            <publishTf>true</publishTf>
-            <publishOdom>true</publishOdom>
+            <publishTf>false</publishTf>
+            <publishOdom>false</publishOdom>
         </plugin>
     </gazebo>

File: nav/urdf/robot_core.xacro (robot description, xacro)
@@ -162,9 +162,9 @@
 		<child link="livox_base"/>
 		<!--origin xyz="0.2 0 1.6" rpy="${M_PI/6} 0 0" /-->
-        <origin xyz="0.2 0 1.6" rpy="0 ${M_PI/6} 0" />
+        <origin xyz="0.2 0 1.6" rpy="${M_PI/6} 0 ${M_PI/2}" />
 	</joint>
     <xacro:include filename="$(find realsense2_description)/urdf/_d435.urdf.xacro" />
     <xacro:sensor_d435 name="camera" topics_ns="camera" parent="livox_base" publish_pointcloud="true">
-        <origin xyz="0 -0.2 -0.3" rpy="0 -${M_PI/6} 0" />
+        <origin xyz="0 -0.2 -0.3" rpy="0 -${M_PI/6} -${M_PI/2}" />
     </xacro:sensor_d435>
     <!-- LEFT WHEEL LINK -->
